File: stmboard/stmboard.kicad_pcb (KiCad board)
At the start: 2 copper layers, 0 parts

Commit message: pcb + footprints
Parts:
- added C1: 1u, Capacitor_SMD:C_0603_1608Metric, F.Cu at (211.6, 121.5)
- added C10: 100n, Capacitor_SMD:C_0603_1608Metric, F.Cu at (211.8, 88.1)
- added C11: 100n, Capacitor_SMD:C_0603_1608Metric, F.Cu at (232.6, 99.2)
- added C12: 1u, Capacitor_SMD:C_0603_1608Metric, F.Cu at (232.6, 122.1)
- added C13: 1u, Capacitor_SMD:C_0603_1608Metric, F.Cu at (232.5, 116.0)
- added C14: 100n, Capacitor_SMD:C_0603_1608Metric, F.Cu at (203.6, 112.8)
- added C15: 18p, Capacitor_SMD:C_0603_1608Metric, F.Cu at (198.1, 89.0)
- added C16: 18p, Capacitor_SMD:C_0603_1608Metric, F.Cu at (200.1, 93.1)
- added C17: 18p, Capacitor_SMD:C_0603_1608Metric, F.Cu at (205.2, 84.1)
- added C18: 18p, Capacitor_SMD:C_0603_1608Metric, F.Cu at (201.1, 85.8)
- added C19: 100n, Capacitor_SMD:C_0603_1608Metric, F.Cu at (210.6, 70.2)
- added C2: 1u, Capacitor_SMD:C_0603_1608Metric, F.Cu at (205.2, 121.7)
- added C20: 100n, Capacitor_SMD:C_0603_1608Metric, F.Cu at (186.1, 55.2)
- added C21: 1u, Capacitor_SMD:C_0603_1608Metric, F.Cu at (178.0, 65.5)
- added C22: 1u, Capacitor_SMD:C_0603_1608Metric, F.Cu at (178.0, 59.5)
- added C23: 100n, Capacitor_SMD:C_0603_1608Metric, F.Cu at (220.2, 83.6)
- added C24: 100n, Capacitor_SMD:C_0603_1608Metric, F.Cu at (224.3, 73.6)
- added C25: 100n, Capacitor_SMD:C_0603_1608Metric, F.Cu at (218.6, 83.6)
- added C26: 100n, Capacitor_SMD:C_0603_1608Metric, F.Cu at (229.5, 86.9)
- added C27: 1u, Capacitor_SMD:C_0603_1608Metric, F.Cu at (230.2, 81.3)
- added C28: 1u, Capacitor_SMD:C_0603_1608Metric, F.Cu at (229.5, 88.7)
- added C29: 100n, Capacitor_SMD:C_0603_1608Metric, F.Cu at (189.1, 77.4)
- added C3: 100n, Capacitor_SMD:C_0603_1608Metric, F.Cu at (208.0, 90.4)
- added C30: 100n, Capacitor_SMD:C_0603_1608Metric, F.Cu at (206.5, 76.6)
- added C31: 100n, Capacitor_SMD:C_0603_1608Metric, F.Cu at (206.5, 78.1)
- added C4: 100n, Capacitor_SMD:C_0603_1608Metric, F.Cu at (208.0, 92.0)
- added C5: 100n, Capacitor_SMD:C_0603_1608Metric, F.Cu at (204.5, 110.4)
- added C6: 100n, Capacitor_SMD:C_0603_1608Metric, F.Cu at (217.7, 100.7)
- added C7: 100n, Capacitor_SMD:C_0603_1608Metric, F.Cu at (197.7, 98.5)
- added C8: 4.7u, Capacitor_SMD:C_0603_1608Metric, F.Cu at (195.4, 100.8)
- added C9: 1u, Capacitor_SMD:C_0603_1608Metric, F.Cu at (196.6, 99.7)
- added D1: LED, LED_SMD:LED_0603_1608Metric, F.Cu at (206.8, 125.0)
- added D2: LED, LED_SMD:LED_0603_1608Metric, F.Cu at (206.2, 88.9)
- added D3: TX, LED_SMD:LED_0603_1608Metric, F.Cu at (210.1, 115.6)
- added D4: RX, LED_SMD:LED_0603_1608Metric, F.Cu at (215.4, 111.2)
- added J1: USB_C_Receptacle_USB2.0_14P, Connector_USB:USB_C_Receptacle_GCT_USB4105-xx-A_16P_TopMnt_Horizontal, F.Cu at (215.3, 128.3)
- added J2: Conn_02x05_Odd_Even, Connector_PinHeader_2.54mm:PinHeader_2x05_P2.54mm_Vertical, F.Cu at (235.5, 107.4)
- added J3: USB_C_Receptacle_USB2.0_14P, Connector_USB:USB_C_Receptacle_GCT_USB4105-xx-A_16P_TopMnt_Horizontal, F.Cu at (228.2, 128.3)
- added J4: Conn_01x20_Socket, Connector_PinHeader_2.54mm:PinHeader_1x20_P2.54mm_Vertical, F.Cu at (245.8, 76.8)
- added J5: Conn_01x20_Socket, Connector_PinHeader_2.54mm:PinHeader_1x20_P2.54mm_Vertical, F.Cu at (169.4, 77.2)
- added J6: USB_C_Receptacle_USB2.0_14P, Connector_USB:USB_C_Receptacle_GCT_USB4105-xx-A_16P_TopMnt_Horizontal, F.Cu at (171.3, 68.7)
- added J7: Micro_SD_Card, Connector_Card:microSD_HC_Molex_47219-2001, B.Cu at (230.8, 59.5)
- added J8: Conn_01x04, Connector_PinSocket_2.54mm:PinSocket_1x04_P2.54mm_Vertical, F.Cu at (245.8, 63.6)
- added LS1: Speaker, STM:BUZ-SMD_4P-L13.0-W13.0-P11.4-BL, F.Cu at (189.5, 86.9)
- added MK1: SPH0645LM4H, Sensor_Audio:Knowles_SPH0645LM4H-6_3.5x2.65mm, F.Cu at (202.9, 76.1)
- added R1: 5.1k, Resistor_SMD:R_0402_1005Metric, F.Cu at (217.6, 121.9)
- added R10: 270, Resistor_SMD:R_0402_1005Metric, F.Cu at (211.5, 116.1)
- added R11: 270, Resistor_SMD:R_0402_1005Metric, F.Cu at (213.5, 112.6)
- added R12: 10k, Resistor_SMD:R_0402_1005Metric, F.Cu at (229.0, 102.6)
- added R13: 10k, Resistor_SMD:R_0402_1005Metric, F.Cu at (198.3, 112.3)
- added R14: 10k, Resistor_SMD:R_0402_1005Metric, F.Cu at (210.5, 72.2)
- added R15: 10k, Resistor_SMD:R_0402_1005Metric, F.Cu at (187.5, 55.5)
- added R16: 5.1k, Resistor_SMD:R_0402_1005Metric, F.Cu at (178.1, 70.4)
- added R17: 5.1k, Resistor_SMD:R_0402_1005Metric, F.Cu at (178.2, 67.0)
- added R18: 10k, Resistor_SMD:R_0402_1005Metric, B.Cu at (215.1, 61.8)
- added R19: 10k, Resistor_SMD:R_0402_1005Metric, F.Cu at (232.9, 55.1)
- added R2: 5.1k, Resistor_SMD:R_0402_1005Metric, F.Cu at (213.3, 121.9)
- added R20: 10k, Resistor_SMD:R_0402_1005Metric, B.Cu at (193.6, 62.5)
- added R21: 10k, Resistor_SMD:R_0402_1005Metric, B.Cu at (212.4, 55.8)
- added R22: 10k, Resistor_SMD:R_0402_1005Metric, B.Cu at (193.6, 57.4)
- added R23: 10k, Resistor_SMD:R_0402_1005Metric, F.Cu at (200.5, 76.1)
- added R3: 10k, Resistor_SMD:R_0402_1005Metric, F.Cu at (216.8, 88.3)
- added R4: 5.1k, Resistor_SMD:R_0402_1005Metric, F.Cu at (230.0, 122.3)
- added R5: 5.1k, Resistor_SMD:R_0402_1005Metric, F.Cu at (226.5, 122.3)
- added R6: 27k, Resistor_SMD:R_0402_1005Metric, F.Cu at (218.3, 115.4)
- added R7: 10k, Resistor_SMD:R_0402_1005Metric, F.Cu at (218.3, 114.4)
- added R8: 1k, Resistor_SMD:R_0402_1005Metric, F.Cu at (205.2, 125.3)
- added R9: 1k, Resistor_SMD:R_0402_1005Metric, F.Cu at (205.2, 90.8)
- added SW1: BOOT0, STM:KEY-SMD_L4.0-W3.0-LS4.9-1, F.Cu at (214.4, 86.7)
- added SW2: NRST, STM:KEY-SMD_L4.0-W3.0-LS4.9-1, F.Cu at (227.3, 100.0)
- added SW3: BOOT, STM:KEY-SMD_L4.0-W3.0-LS4.9-1, F.Cu at (210.4, 76.0)
- added SW4: BOOT, STM:KEY-SMD_L4.0-W3.0-LS4.9-1, F.Cu at (186.7, 59.9)
- added U1: STM32F411RCTx, Package_QFP:LQFP-64_10x10mm_P0.5mm, F.Cu at (207.5, 101.4)
- added U10: MAX98357A, Package_DFN_QFN:TQFN-16-1EP_3x3mm_P0.5mm_EP1.23x1.23mm, F.Cu at (193.9, 76.3)
- added U2: ESP32-S3-WROOM-1, RF_Module:ESP32-S3-WROOM-1, F.Cu at (199.0, 58.9)
- added U3: AP2112K-3.3, Package_TO_SOT_SMD:SOT-23-5, F.Cu at (208.2, 121.5)
- added U4: AP2112K-3.3, Package_TO_SOT_SMD:SOT-23-5, F.Cu at (232.7, 119.1)
- added U5: CP2102N-Axx-xQFN20, Package_DFN_QFN:SiliconLabs_QFN-20-1EP_3x3mm_P0.5mm_EP1.8x1.8mm, F.Cu at (214.8, 115.6)
- added U6: AP2112K-3.3, Package_TO_SOT_SMD:SOT-23-5, F.Cu at (178.1, 62.6)
- added U7: ICM-20948, Sensor_Motion:InvenSense_QFN-24_3x3mm_P0.4mm, F.Cu at (224.3, 77.8)
- added U8: TXB0102DCT, Package_SO:TSSOP-8_3x3mm_P0.65mm, F.Cu at (224.4, 83.9)
- added U9: AP2112K-1.8, Package_TO_SOT_SMD:SOT-23-5, F.Cu at (229.8, 84.0)
- added Y1: 25MHz, Crystal:Crystal_SMD_Abracon_ABM8G-4Pin_3.2x2.5mm, F.Cu at (201.2, 89.2)
- added Y2: 32.768KHz, Crystal:Crystal_SMD_Abracon_ABM8G-4Pin_3.2x2.5mm, F.Cu at (201.2, 83.0)
Routing:
- net /NRST: track 0.00 -> 123.0 mm, vias 0 -> 5
- net /SWDIO: track 0.00 -> 105.8 mm, vias 0 -> 1
- net GND: track 0.00 -> 93.7 mm, vias 0 -> 17
- net +3V3: track 0.00 -> 86.9 mm, vias 0 -> 44
- net /PB6: track 0.00 -> 84.4 mm, vias 0 -> 2
- net /BOOT0: track 0.00 -> 77.6 mm, vias 0 -> 3
- net /PB7: track 0.00 -> 76.9 mm, vias 0 -> 2
- net /SWCLK: track 0.00 -> 71.0 mm, vias 0 -> 4
- net /PC3: track 0.00 -> 64.7 mm, vias 0 -> 4
- net /PC2: track 0.00 -> 63.3 mm, vias 0 -> 4
- net /PA15: track 0.00 -> 59.8 mm
- net /PC10: track 0.00 -> 58.1 mm
- net /PA8: track 0.00 -> 56.8 mm
- net /PC11: track 0.00 -> 56.6 mm
- net /PC9: track 0.00 -> 54.9 mm
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- added copper zone on B.Cu, net +3V3
- added copper zone on F.Cu, net GND
Other:
- board outline added: 80 x 80 mm
