File: stmboard/stmboard.kicad_sch (KiCad schematic)
At the start: 48 parts, among them J1 USB_C_Receptacle_USB2.0_14P, J2 Conn_02x05_Odd_Even, J3 USB_C_Receptacle_USB2.0_14P, J4 Conn_01x20_Socket, J5 Conn_01x20_Socket, SW1 BOOT0, SW2 NRST, U1 STM32F411RCTx, U3 AP2112K-3.3, U4 AP2112K-3.3, U5 CP2102N-Axx-xQFN20, Y1 25MHz, Y2 32.768KHz

Commit message: workingon schematic crystals ldos usb cp2102 leds
Parts:
- removed J2: Conn_02x05_Odd_Even, Connector_PinHeader_2.54mm:PinHeader_2x05_P2.54mm_Vertical, symbol Connector_Generic:Conn_02x05_Odd_Even
- removed J4, J5: Conn_01x20_Socket, Connector_PinHeader_2.54mm:PinHeader_1x20_P2.54mm_Vertical, symbol Connector:Conn_01x20_Socket
- C1, C10, C11, C12, C13, C14, C15, C16, C17, C18, C2, C3, C4, C5, C6, C7, C8, C9: footprint Capacitor_SMD:C_0805_2012Metric -> Capacitor_SMD:C_0603_1608Metric
- D1, D2, D3, D4: footprint LED_SMD:LED_0805_2012Metric -> LED_SMD:LED_0603_1608Metric
- R1, R10, R11, R12, R13, R2, R3, R4, R5, R6, R7, R8, R9: footprint Resistor_SMD:R_0805_2012Metric -> Resistor_SMD:R_0402_1005Metric
- SW1, SW2: footprint Button_Switch_SMD:SW_Push_1P1T_NO_CK_KMR2 -> STM:KEY-SMD_L4.0-W3.0-LS4.9-1
Connections:
- net PA2 renamed TX1
- net PA3 renamed RX1
- no-connect marks 12 -> 11
Other:
- moved on the sheet: C1, C10, C11, C12, C13, C14, C15, C16, C17, C18, C2, C3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

Commit message: sd card sdmmc esp32
Parts:
- added C19, C20: 100n, Capacitor_SMD:C_0603_1608Metric, symbol Device:C
- added C21, C22: 1u, Capacitor_SMD:C_0603_1608Metric, symbol Device:C
- added J2: Conn_02x05_Odd_Even, Connector_PinHeader_2.54mm:PinHeader_2x05_P2.54mm_Vertical, symbol Connector_Generic:Conn_02x05_Odd_Even
- added J4, J5: Conn_01x20_Socket, Connector_PinHeader_2.54mm:PinHeader_1x20_P2.54mm_Vertical, symbol Connector:Conn_01x20_Socket
- added J6: USB_C_Receptacle_USB2.0_14P, Connector_USB:USB_C_Receptacle_GCT_USB4105-xx-A_16P_TopMnt_Horizontal, symbol Connector:USB_C_Receptacle_USB2.0_14P
- added J7: Micro_SD_Card, symbol Connector:Micro_SD_Card
- added R14, R15, R18, R19, R20, R21, R22: 10k, Resistor_SMD:R_0402_1005Metric, symbol Device:R
- added R16, R17: 5.1k, Resistor_SMD:R_0402_1005Metric, symbol Device:R
- added SW3, SW4: BOOT, STM:KEY-SMD_L4.0-W3.0-LS4.9-1, symbol Switch:SW_Push
- added U2: ESP32-S3-WROOM-1, RF_Module:ESP32-S3-WROOM-1, symbol RF_Module:ESP32-S3-WROOM-1
- added U6: AP2112K-3.3, Package_TO_SOT_SMD:SOT-23-5, symbol Regulator_Linear:AP2112K-3.3
Connections:
- net +3V3: now also C22.1, J2.7 (Pin_7), J2.8 (Pin_8), J7.4 (VDD), R14.1, R15.1, R18.1, R19.1, R20.1, R21.1, R22.1, U2.2 (3V3), U6.5 (VOUT)
- net BOOT0: now also U2.31 (IO38)
- net GND: now also C19.2, C20.2, C21.2, C22.2, J2.5 (Pin_5), J2.6 (Pin_6), J6.A1 (GND), J6.A12 (GND), J6.B1 (GND), J6.B12 (GND), J6.SH (SHIELD), J7.6 (VSS), J7.SH (SHIELD), R16.2, R17.1, SW3.1, SW4.1, U2.1 (GND), U2.40 (GND), U2.41 (GND), U6.2 (GND)
- net NRST: now also J2.1 (Pin_1), U2.32 (IO39)
- net RX1: now also U2.37 (TXD0)
- net SWCLK: now also J2.2 (Pin_2)
- net SWDIO: now also J2.4 (Pin_4), U2.33 (IO40)
- net TX1: now also U2.36 (RXD0)
- net VBUS: now also J2.10 (Pin_10), J2.9 (Pin_9)
- new net: C19.1, R14.2, SW3.2, U2.27 (IO0)
- new net: C20.1, R15.2, SW4.2, U2.3 (EN)
- new net: C21.1, J6.A4 (VBUS), J6.A9 (VBUS), J6.B4 (VBUS), J6.B9 (VBUS), U6.1 (VIN), U6.3 (EN)
- new net: J6.A5 (CC1), R17.2
- new net: J6.B5 (CC2), R16.1
- new net CLK: J7.5 (CLK), U2.22 (IO14)
- new net CMD: J7.3 (CMD), R20.2, U2.8 (IO15)
- new net DAT0: J7.7 (DAT0), R21.2, U2.38 (IO2)
- new net DAT1: J7.8 (DAT1), R22.2, U2.4 (IO4)
- new net DAT2: J7.1 (DAT2), R18.2, U2.20 (IO12)
- new net DAT3: J7.2 (DAT3/CD), R19.2, U2.21 (IO13)
- new net D_{1}+: J6.A6 (D+), J6.B6 (D+), U2.14 (USB_D+)
- new net D_{1}-: J6.A7 (D-), J6.B7 (D-), U2.13 (USB_D-)
- new net SCLK: U2.34 (IO41)
- no-connect marks 11 -> 12

Commit message: 9 dof + voltage reg
Parts:
- added C23, C24, C25, C26: 100n, Capacitor_SMD:C_0603_1608Metric, symbol Device:C
- added C27, C28: 1u, Capacitor_SMD:C_0603_1608Metric, symbol Device:C
- added J8: Conn_01x04, symbol Connector_Generic:Conn_01x04
- added U7: ICM-20948, Sensor_Motion:InvenSense_QFN-24_3x3mm_P0.4mm, symbol Sensor_Motion:ICM-20948
- added U8: TXB0102DCT, Package_SO:TSSOP-8_3x3mm_P0.65mm, symbol Logic_LevelTranslator:TXB0102DCT
- added U9: AP2112K-1.8, Package_TO_SOT_SMD:SOT-23-5, symbol Regulator_Linear:AP2112K-1.8
Connections:
- net +3V3: now also C23.1, C25.1, C27.1, J8.2 (Pin_2), U7.13 (VDD), U8.7 (VCCB), U9.1 (VIN), U9.3 (EN)
- net GND: now also C23.2, C24.2, C25.2, C26.2, C27.2, C28.2, J8.1 (Pin_1), U7.18 (GND), U7.20 (GND), U7.9 (SDO/AD0), U8.2 (GND), U8.6 (OE), U9.2 (GND)
- net PB6: now also J8.3 (Pin_3), U8.1 (B2)
- net PB7: now also J8.4 (Pin_4), U8.8 (B1)
- new net: C24.1, U7.10 (REGOUT)
- new net +1V8: C26.1, C28.1, U7.8 (VDDIO), U8.3 (VCCA), U9.5 (VOUT)
- new net SCL_{1V8}: U7.23 (SCL/SCLK), U8.4 (A2)
- new net SDA_{1V8}: U7.24 (SDA/SDI), U8.5 (A1)
- no-connect marks 12 -> 17
Other:
- moved on the sheet: C3, C4, C5, C6, C7, C8, C9

Commit message: speaker
Parts:
- added C29: 100n, Capacitor_SMD:C_0603_1608Metric, symbol Device:C
- added LS1: Speaker, symbol Device:Speaker
- added U10: MAX98357A, Package_DFN_QFN:TQFN-16-1EP_3x3mm_P0.5mm_EP1.23x1.23mm, symbol Audio:MAX98357A
Connections:
- net +3V3: now also C29.1, U10.2 (GAIN_SLOT), U10.7 (VDD), U10.8 (VDD)
- net GND: now also C29.2, U10.11 (GND), U10.15 (GND), U10.17 (PAD), U10.3 (GND)
- net FCLK: now reaches U2.16 (IO46)
- net FCLK: now also U10.14 (LRCLK)
- net ~{SD_MODE}: now reaches U2.24 (IO47)
- net ~{SD_MODE}: now also U10.4 (~{SD_MODE})
- net BCLK: now reaches U2.26 (IO45)
- net BCLK: now also U10.16 (BCLK)
- net DIN: now reaches U2.35 (IO42)
- net DIN: now also U10.1 (DIN)
- new net: LS1.2, U10.10 (OUTN)
- new net: LS1.1, U10.9 (OUTP)
Other:
- moved on the sheet: C10, C11, C3, C4, C5, C6, C7, C8, C9, R12, R13, R3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

Commit message: mic + footprints
Parts:
- added C30, C31: 100n, Capacitor_SMD:C_0603_1608Metric, symbol Device:C
- added MK1: SPH0645LM4H, Sensor_Audio:Knowles_SPH0645LM4H-6_3.5x2.65mm, symbol Sensor_Audio:SPH0645LM4H
- added R23: 10k, symbol Device:R
Connections:
- net +3V3: now also C30.1, C31.1, MK1.5 (VDD)
- net GND: now also C30.2, C31.2, MK1.3 (GND), R23.2
- new net: MK1.2 (SEL), R23.1
- new net BCLK2: MK1.4 (BCLK)
- new net DATA: MK1.6 (DATA)
- new net WS: MK1.1 (WS)
Other:
- moved on the sheet: C14, C29, C3, C4, C5, C6, C7, C8, C9, LS1, U1, U10

Commit message: pcb + footprints
Parts:
- J7: footprint (none) -> Connector_Card:microSD_HC_Molex_47219-2001
- J8: footprint (none) -> Connector_PinSocket_2.54mm:PinSocket_1x04_P2.54mm_Vertical
- LS1: footprint (none) -> STM:BUZ-SMD_4P-L13.0-W13.0-P11.4-BL
- R23: footprint (none) -> Resistor_SMD:R_0402_1005Metric
Connections:
- net SCLK is gone; now on net SWCLK: U2.34 (IO41)
- net +3V3: now also J4.1 (Pin_1), J5.2 (Pin_2)
- net BCLK: now also U2.17 (IO9); no longer U2.26 (IO45)
- net BCLK2: now also U2.25 (IO48)
- net BOOT0: now also J5.1 (Pin_1)
- net DATA: now also U2.24 (IO47)
- net DIN: now also U2.16 (IO46); no longer U2.35 (IO42)
- net FCLK: now also U2.18 (IO10); no longer U2.16 (IO46)
- net GND: now also J4.2 (Pin_2), J5.3 (Pin_3)
- net NRST: now also J5.6 (Pin_6)
- net PA15: now also J5.20 (Pin_20)
- net PA4: now also J4.3 (Pin_3)
- net PA5: now also J4.4 (Pin_4)
- net PA6: now also J4.5 (Pin_5)
- net PA7: now also J4.6 (Pin_6)
- net PA8: now also J4.20 (Pin_20)
- net PB0: now also J4.9 (Pin_9)
- net PB1: now also J4.10 (Pin_10)
- net PB10: now also J4.11 (Pin_11)
- net PB12: now also J4.12 (Pin_12)
- net PB13: now also J4.13 (Pin_13)
- net PB14: now also J4.15 (Pin_15)
- net PB15: now also J4.14 (Pin_14)
- net PB3: now also J5.16 (Pin_16)
- net PB4: now also J5.15 (Pin_15)
- net PB5: now also J5.14 (Pin_14)
- net PB6: now also J5.11 (Pin_11)
- net PB7: now also J5.10 (Pin_10)
- net PB8: now also J5.13 (Pin_13)
- net PB9: now also J5.12 (Pin_12)
- net PC0: now also J5.9 (Pin_9)
- net PC1: now also J5.8 (Pin_8)
- net PC10: now also J5.19 (Pin_19)
- net PC11: now also J5.18 (Pin_18)
- net PC12: now also J5.17 (Pin_17)
- net PC2: now also J5.5 (Pin_5)
- net PC3: now also J5.4 (Pin_4)
- net PC4: now also J4.7 (Pin_7)
- net PC5: now also J4.8 (Pin_8)
- net PC6: now also J4.16 (Pin_16)
- net PC7: now also J4.17 (Pin_17)
- net PC8: now also J4.18 (Pin_18)
- net PC9: now also J4.19 (Pin_19)
- net SWDIO: now also J5.7 (Pin_7)
- net WS: now also U2.23 (IO21)
- net ~{SD_MODE}: now also U2.15 (IO3); no longer U2.24 (IO47)
- no-connect marks 17 -> 31
